File: FRA261.kicad_pcb (KiCad board)
At the start: 2 copper layers, 162.7 x 164.1 mm, 68 parts

Commit message: updata
Parts:
- added G***: LOGO, LOGO, F.Cu at (197.6, 49.3)
Other:
- board text added: "ECA"
- board text added: "ECB"
- board text added: "EG1"
- board text added: "EG2"
- board text added: "EG3"
- board text added: "GND"
- board text added: "SCL"
- board text added: "SDA"
- board text added: "Signal"
- board text added: "VCC"

Commit message: updata
Parts:
- Logic_Analyzer1: value Conn_01x04_Female -> Conn_01x05_Female; footprint Connector_PinSocket_2.54mm:PinSocket_1x04_P2.54mm_Vertical -> Connector_PinSocket_2.54mm:PinSocket_1x05_P2.54mm_Vertical
- moved G*** 168.6 mm to (87.2, 176.7)
- moved Logic_Analyzer1 3.00 mm to (118.1, 181.6)
Connections:
- ES1 pad 1: PA10 -> PC10
- ESP32 pad 13: PA3 -> PA10
- ESP32 pad 16: 5V_Nucleo_F411RE -> 5V
- Logic_Analyzer1 pad 4: PA3 -> PA10
- STM32F411RE1 pad 1: unconnected-(STM32F411RE1-Pad1) -> PC10
- STM32F411RE1 pad 18: 5V_Nucleo_F411RE -> unconnected-(STM32F411RE1-Pad18)
- STM32F411RE1 pad 34: unconnected-(STM32F411RE1-Pad34) -> PB0
- STM32F411RE1 pad 75: PA3 -> unconnected-(STM32F411RE1-Pad75)
- SW_PWM1 pad 3: unconnected-(SW_PWM1-Pad3) -> PB0
Routing:
- net PA3: track 227.6 -> 0.00 mm, vias 1 -> 0
- net PC10: track 0.00 -> 159.9 mm, vias 0 -> 5
- net PA10: track 114.5 -> 241.2 mm, vias 3 -> 1
- net 5V_Nucleo_F411RE: track 66.7 -> 0.00 mm, vias 2 -> 0
- net PB0: track 0.00 -> 49.1 mm, vias 0 -> 2
- net 5V: track 414.5 -> 420.1 mm
- net sw6: track 63.6 -> 61.8 mm
- net sw5: track 57.0 -> 55.2 mm
- net sw2: track 134.5 -> 133.9 mm
- removed copper zone on B.Cu, net GND
- removed copper zone on F.Cu, net GND
