File: FRA261.kicad_sch (KiCad schematic)
At the start: 68 parts

Commit message: updata
Parts:
- removed Logic_Analyzer1: Conn_01x04_Female, Connector_PinSocket_2.54mm:PinSocket_1x04_P2.54mm_Vertical, symbol Connector:Conn_01x04_Female
- added Logic_Analyzer1: Conn_01x05_Female, Connector_PinSocket_2.54mm:PinSocket_1x05_P2.54mm_Vertical, symbol Connector:Conn_01x05_Female
Connections:
- net 5V: now also ESP32.16 (VIN)
- net GND: now also Logic_Analyzer1.5 (Pin_5)
- net PA10: now also ESP32.13 (TX0), Logic_Analyzer1.4 (Pin_4); no longer ES1.1 (A)
- net sw2: now also Logic_Analyzer1.1 (Pin_1)
- net sw5: now also Logic_Analyzer1.2 (Pin_2)
- net sw6: now also Logic_Analyzer1.3 (Pin_3)
- net PC10: now reaches STM32F411RE1.1 (PC10)
- net PC10: now also ES1.1 (A)
- net PB0: now reaches STM32F411RE1.34 (PB0)
- net PB0: now also SW_PWM1.3 (B)
- net 5V_Nucleo_F411RE: no longer names the net of STM32F411RE1.18 (+5V)
- net 5V_Nucleo_F411RE: no longer ESP32.16 (VIN)
- net PA3: no longer names the net of STM32F411RE1.75 (PA3)
- net PA3: no longer ESP32.13 (TX0)
- no-connect marks 91 -> 90
